File: fmr50nbx2/fdd_adapter/part1/26_to_26_pin_adapter.kicad_pcb (KiCad board)
At the start: 2 copper layers, 68.9 x 11.5 mm, 2 parts, among them J1 Conn_01x26_Female, J2 Conn_01x26_Female

Commit message: Add files via upload
Parts:
- J1: footprint msx cartridge:fdd_26_pin_insert -> Connector:fdd_26_pin_insert_both_sides
- moved J1 31.2 mm to (96.4, 64.2), turned to 0 degrees
- moved J2 1.00 mm to (69.2, 58.1)
Routing:
- net VCC: track 97.6 -> 45.6 mm
- net GND: track 76.7 -> 60.6 mm
- net Net-(J1-Pad18): track 12.9 -> 9.91 mm
- net Net-(J1-Pad16): track 14.0 -> 12.4 mm
- net Net-(J1-Pad6): track 24.9 -> 25.3 mm, vias 1 -> 0
- net Net-(J1-Pad10): track 19.7 -> 20.0 mm, vias 1 -> 0
- net Net-(J1-Pad8): track 22.3 -> 22.6 mm, vias 1 -> 0
- net Net-(J1-Pad9): track 21.1 -> 21.3 mm, vias 1 -> 0
- net Net-(J1-Pad20): vias 1 -> 0
Other:
- board size 68.9 x 11.5 mm -> 67.4 x 10 mm
- net class power: trace_width 1 -> 0.75; via_dia 1.6 -> 1.5
- net class power2 added: clearance 0.3, trace_width 0.5, via_dia 1, via_drill 0.5
