File: fmr50nbx2/fdd_adapter/part1/26_to_26_pin_adapter.sch (KiCad schematic (older format))
At the start: 2 parts, among them J1 Conn_01x26_Female, J2 Conn_01x26_Female

Commit message: Add files via upload
Parts:
- J1: footprint msx cartridge:fdd_26_pin_insert -> Connector:fdd_26_pin_insert_both_sides
Changed lines of the file:
@@
 F 0 "J1" H 2178 2476 50  0000 L CNN
 F 1 "Conn_01x26_Female" H 2178 2385 50  0000 L CNN
-F 2 "msx cartridge:fdd_26_pin_insert" H 2150 2500 50  0001 C CNN
+F 2 "Connector:fdd_26_pin_insert_both_sides" H 2150 2500 50  0001 C CNN
 F 3 "~" H 2150 2500 50  0001 C CNN
 	1    2150 2500
