File: 1.25mm_to_1mm_adapter/26_to_26_pin_adapter.kicad_pcb (KiCad board)
At the start: 2 copper layers, 33.6 x 11.7 mm, 2 parts, among them J1 Conn_01x26_Female, J2 Conn_01x26_Female

Commit message: Add files via upload
Other:
- board size 33.6 x 11.7 mm -> 33.6 x 12.4 mm
Changed lines of the file:
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@@
     (pad 1 thru_hole circle (at 0 -1.25) (size 0.9 0.9) (drill 0.45) (layers *.Cu *.Mask)
       (net 19 VCC))
-    (pad 26 connect rect (at 31.25 -0.127) (size 0.75 3) (layers F.Cu B.Mask)
+    (pad 26 connect rect (at 31.25 -0.127) (size 0.75 3) (layers F.Cu F.Mask)
       (net 1 "Net-(J1-Pad26)"))
-    (pad 25 connect rect (at 30 -0.127) (size 0.75 3) (layers F.Cu B.Mask)
+    (pad 25 connect rect (at 30 -0.127) (size 0.75 3) (layers F.Cu F.Mask)
       (net 18 GND))
-    (pad 24 connect rect (at 28.75 -0.127) (size 0.75 3) (layers F.Cu B.Mask)
+    (pad 24 connect rect (at 28.75 -0.127) (size 0.75 3) (layers F.Cu F.Mask)
       (net 2 "Net-(J1-Pad24)"))
-    (pad 23 connect rect (at 27.5 -0.127) (size 0.75 3) (layers F.Cu B.Mask)
+    (pad 23 connect rect (at 27.5 -0.127) (size 0.75 3) (layers F.Cu F.Mask)
       (net 18 GND))
-    (pad 22 connect rect (at 26.25 -0.127) (size 0.75 3) (layers F.Cu B.Mask)
+    (pad 22 connect rect (at 26.25 -0.127) (size 0.75 3) (layers F.Cu F.Mask)
       (net 17 "Net-(J1-Pad22)"))
-    (pad 21 connect rect (at 25 -0.127) (size 0.75 3) (layers F.Cu B.Mask)
+    (pad 21 connect rect (at 25 -0.127) (size 0.75 3) (layers F.Cu F.Mask)
       (net 18 GND))
-    (pad 20 connect rect (at 23.75 -0.127) (size 0.75 3) (layers F.Cu B.Mask)
+    (pad 20 connect rect (at 23.75 -0.127) (size 0.75 3) (layers F.Cu F.Mask)
       (net 16 "Net-(J1-Pad20)"))
-    (pad 19 connect rect (at 22.5 -0.127) (size 0.75 3) (layers F.Cu B.Mask)
+    (pad 19 connect rect (at 22.5 -0.127) (size 0.75 3) (layers F.Cu F.Mask)
       (net 18 GND))
-    (pad 18 connect rect (at 21.25 -0.127) (size 0.75 3) (layers F.Cu B.Mask)
+    (pad 18 connect rect (at 21.25 -0.127) (size 0.75 3) (layers F.Cu F.Mask)
       (net 15 "Net-(J1-Pad18)"))
-    (pad 17 connect rect (at 20 -0.127) (size 0.75 3) (layers F.Cu B.Mask)
+    (pad 17 connect rect (at 20 -0.127) (size 0.75 3) (layers F.Cu F.Mask)
       (net 18 GND))
-    (pad 16 connect rect (at 18.75 -0.127) (size 0.75 3) (layers F.Cu B.Mask)
+    (pad 16 connect rect (at 18.75 -0.127) (size 0.75 3) (layers F.Cu F.Mask)
       (net 14 "Net-(J1-Pad16)"))
-    (pad 15 connect rect (at 17.5 -0.127) (size 0.75 3) (layers F.Cu B.Mask)
+    (pad 15 connect rect (at 17.5 -0.127) (size 0.75 3) (layers F.Cu F.Mask)
       (net 18 GND))
-    (pad 14 connect rect (at 16.25 -0.127) (size 0.75 3) (layers F.Cu B.Mask)
+    (pad 14 connect rect (at 16.25 -0.127) (size 0.75 3) (layers F.Cu F.Mask)
       (net 13 "Net-(J1-Pad14)"))
-    (pad 13 connect rect (at 15 -0.127) (size 0.75 3) (layers F.Cu B.Mask)
+    (pad 13 connect rect (at 15 -0.127) (size 0.75 3) (layers F.Cu F.Mask)
       (net 12 "Net-(J1-Pad13)"))
-    (pad 12 connect rect (at 13.75 -0.127) (size 0.75 3) (layers F.Cu B.Mask)
+    (pad 12 connect rect (at 13.75 -0.127) (size 0.75 3) (layers F.Cu F.Mask)
       (net 11 "Net-(J1-Pad12)"))
-    (pad 11 connect rect (at 12.5 -0.127) (size 0.75 3) (layers F.Cu B.Mask)
+    (pad 11 connect rect (at 12.5 -0.127) (size 0.75 3) (layers F.Cu F.Mask)
       (net 10 "Net-(J1-Pad11)"))
-    (pad 10 connect rect (at 11.25 -0.127) (size 0.75 3) (layers F.Cu B.Mask)
+    (pad 10 connect rect (at 11.25 -0.127) (size 0.75 3) (layers F.Cu F.Mask)
       (net 9 "Net-(J1-Pad10)"))
-    (pad 9 connect rect (at 10 -0.127) (size 0.75 3) (layers F.Cu B.Mask)
+    (pad 9 connect rect (at 10 -0.127) (size 0.75 3) (layers F.Cu F.Mask)
       (net 8 "Net-(J1-Pad9)"))
-    (pad 8 connect rect (at 8.75 -0.127) (size 0.75 3) (layers F.Cu B.Mask)
+    (pad 8 connect rect (at 8.75 -0.127) (size 0.75 3) (layers F.Cu F.Mask)
       (net 7 "Net-(J1-Pad8)"))
-    (pad 7 connect rect (at 7.5 -0.127) (size 0.75 3) (layers F.Cu B.Mask)
+    (pad 7 connect rect (at 7.5 -0.127) (size 0.75 3) (layers F.Cu F.Mask)
       (net 6 "Net-(J1-Pad7)"))
-    (pad 6 connect rect (at 6.25 -0.127) (size 0.75 3) (layers F.Cu B.Mask)
+    (pad 6 connect rect (at 6.25 -0.127) (size 0.75 3) (layers F.Cu F.Mask)
       (net 5 "Net-(J1-Pad6)"))
-    (pad 5 connect rect (at 5 -0.127) (size 0.75 3) (layers F.Cu B.Mask)
+    (pad 5 connect rect (at 5 -0.127) (size 0.75 3) (layers F.Cu F.Mask)
       (net 19 VCC))
-    (pad 4 connect rect (at 3.75 -0.127) (size 0.75 3) (layers F.Cu B.Mask)
+    (pad 4 connect rect (at 3.75 -0.127) (size 0.75 3) (layers F.Cu F.Mask)
       (net 4 "Net-(J1-Pad4)"))
-    (pad 3 connect rect (at 2.5 -0.127) (size 0.75 3) (layers F.Cu B.Mask)
+    (pad 3 connect rect (at 2.5 -0.127) (size 0.75 3) (layers F.Cu F.Mask)
       (net 19 VCC))
-    (pad 2 connect rect (at 1.25 -0.127) (size 0.75 3) (layers F.Cu B.Mask)
+    (pad 2 connect rect (at 1.25 -0.127) (size 0.75 3) (layers F.Cu F.Mask)
       (net 3 "Net-(J1-Pad2)"))
-    (pad 1 connect rect (at 0 -0.127) (size 0.75 3) (layers F.Cu B.Mask)
+    (pad 1 connect rect (at 0 -0.127) (size 0.75 3) (layers F.Cu F.Mask)
       (net 19 VCC))
     (pad 1 connect rect (at 0 -0.127) (size 0.75 3) (layers B.Cu B.Mask)
@@
   )
   (gr_line (start 128.843 66) (end 95.193 66) (layer Edge.Cuts) (width 0.05))
-  (gr_line (start 95.193 66) (end 95.193 54.3) (layer Edge.Cuts) (width 0.05))
-  (gr_line (start 128.843 54.3) (end 128.843 66) (layer Edge.Cuts) (width 0.05))
-  (gr_line (start 95.193 54.3) (end 128.843 54.3) (layer Edge.Cuts) (width 0.05))
+  (gr_line (start 95.193 66) (end 95.193 53.6) (layer Edge.Cuts) (width 0.05))
+  (gr_line (start 128.843 53.6) (end 128.843 66) (layer Edge.Cuts) (width 0.05))
+  (gr_line (start 95.193 53.6) (end 128.843 53.6) (layer Edge.Cuts) (width 0.05))
   (segment (start 127.643 63.139) (end 127.643 57.3712) (width 0.25) (layer B.Cu) (net 1))
   (segment (start 127.643 57.3712) (end 125.88 55.6082) (width 0.25) (layer B.Cu) (net 1))
